Commit message: apply xml formatter

File: urdf/actuator.xacro (robot description, xacro)
@@ -8,6 +8,6 @@
     </joint>
     <actuator name="steering_left_front_motor">
-       <hardwareInterface>hardware_interface/EffortJointInterface</hardwareInterface>
-       <mechanismReduction>1</mechanismReduction>
+      <hardwareInterface>hardware_interface/EffortJointInterface</hardwareInterface>
+      <mechanismReduction>1</mechanismReduction>
     </actuator>
   </transmission>
@@ -18,6 +18,6 @@
     </joint>
     <actuator name="steering_right_front_motor">
-       <hardwareInterface>hardware_interface/EffortJointInterface</hardwareInterface>
-       <mechanismReduction>1</mechanismReduction>
+      <hardwareInterface>hardware_interface/EffortJointInterface</hardwareInterface>
+      <mechanismReduction>1</mechanismReduction>
     </actuator>
   </transmission>
@@ -29,6 +29,6 @@
     </joint>
     <actuator name="wheel_left_rear_motor">
-       <hardwareInterface>hardware_interface/VelocityJointInterface</hardwareInterface>
-       <mechanismReduction>1</mechanismReduction>
+      <hardwareInterface>hardware_interface/VelocityJointInterface</hardwareInterface>
+      <mechanismReduction>1</mechanismReduction>
     </actuator>
   </transmission>
@@ -39,6 +39,6 @@
     </joint>
     <actuator name="wheel_right_rear_motor">
-       <hardwareInterface>hardware_interface/VelocityJointInterface</hardwareInterface>
-       <mechanismReduction>1</mechanismReduction>
+      <hardwareInterface>hardware_interface/VelocityJointInterface</hardwareInterface>
+      <mechanismReduction>1</mechanismReduction>
     </actuator>
   </transmission>

File: urdf/wheel.xacro (robot description, xacro)
@@ -7,5 +7,5 @@
       <origin rpy="0 0 ${pi/2}" xyz="${x} ${y} 0"/>
       <parent link="${parent}"/>
-      <child  link="${suffix}_link"/>
+      <child link="${suffix}_link"/>
       <axis xyz="1 0 0"/>
       <dynamics damping="0.1"/>
@@ -26,5 +26,5 @@
         <origin xyz="0 0 0" rpy="0 0 0"/>
         <mass value="${mass}"/>
-        <inertia ixx="${mass*radius*radius/2}"  ixy="0"  ixz="0" iyy="${radius*radius*mass/4+width*width*mass/12}" iyz="0" izz="${radius*radius*mass/4+width*width*mass/12}" />
+        <inertia ixx="${mass*radius*radius/2}" ixy="0" ixz="0" iyy="${radius*radius*mass/4+width*width*mass/12}" iyz="0" izz="${radius*radius*mass/4+width*width*mass/12}" />
       </inertial>
       <collision>
