Commit message: fixed tf frame

File: urdf/body.xacro (robot description, xacro)
@@ -1,9 +1,9 @@
 <?xml version="1.0"?>
 <robot xmlns:xacro="http://ros.org/wiki/xacro">
-  <xacro:macro name="body_macro" params="suffix parent wheel_radius wheel_base vehicle_mass vehicle_mass_height vehicle_width vehicle_length vehicle_height">
+  <xacro:macro name="body_macro" params="suffix parent wheel_base vehicle_mass vehicle_mass_height vehicle_width vehicle_length vehicle_height">
   <xacro:property name="pi" value="3.1415926835897931" />
     <joint name="${suffix}_joint" type="fixed">
       <parent link="${parent}"/>
-      <origin rpy="0 0 0" xyz="0 0 ${wheel_radius}"/>
+      <origin rpy="0 0 0" xyz="0 0 0"/>
       <child  link="${suffix}_link"/>
     </joint>

File: urdf/vehicle.xacro (robot description, xacro)
@@ -10,5 +10,5 @@
   <xacro:arg name="gpu" default="false"/>
   <xacro:property name="pi" value="3.1415926835897931"/>
-  <link name="base_footprint"/>
+  <link name="base_link"/>
   <!-- ================ vehicle ================ -->
   <!-- load parameter -->
@@ -25,7 +25,6 @@
   <xacro:property name="vehicle_mass_height" value="0.5"/>
   <!-- body-->
-  <xacro:body_macro suffix="base"
-                    parent="base_footprint"
-                    wheel_radius="${wheel_radius}"
+  <xacro:body_macro suffix="base_body"
+                    parent="base_link"
                     wheel_base="${wheel_base}"
                     vehicle_mass="${vehicle_mass}"
@@ -34,4 +33,11 @@
                     vehicle_width="${vehicle_width}"
                     vehicle_height="${vehicle_height}"/>
+  <joint name="base_footprint_joint" type="fixed">
+    <parent link="base_link"/>
+    <origin rpy="0 0 0" xyz="0 0 ${-wheel_radius}"/>
+    <child  link="base_footprint"/>
+  </joint>
+  <link name="base_footprint">
+  </link>
   <!-- steering-->
   <xacro:steering_link_macro suffix="steering_front" parent="base_link" x="${wheel_base}" y="0"/>

Commit message: update tf frame

File: urdf/body.xacro (robot description, xacro)
@@ -1,9 +1,9 @@
 <?xml version="1.0"?>
 <robot xmlns:xacro="http://ros.org/wiki/xacro">
-  <xacro:macro name="body_macro" params="suffix parent wheel_base vehicle_mass vehicle_mass_height vehicle_width vehicle_length vehicle_height">
+  <xacro:macro name="body_macro" params="suffix parent wheel_radius wheel_base vehicle_mass vehicle_mass_height vehicle_width vehicle_length vehicle_height">
   <xacro:property name="pi" value="3.1415926835897931" />
     <joint name="${suffix}_joint" type="fixed">
       <parent link="${parent}"/>
-      <origin rpy="0 0 0" xyz="0 0 0"/>
+      <origin rpy="0 0 0" xyz="0 0 ${wheel_radius}"/>
       <child  link="${suffix}_link"/>
     </joint>

File: urdf/vehicle.xacro (robot description, xacro)
@@ -27,4 +27,5 @@
   <xacro:body_macro suffix="base_body"
                     parent="base_link"
+                    wheel_radius="${wheel_radius}"
                     wheel_base="${wheel_base}"
                     vehicle_mass="${vehicle_mass}"
@@ -33,13 +34,6 @@
                     vehicle_width="${vehicle_width}"
                     vehicle_height="${vehicle_height}"/>
-  <joint name="base_footprint_joint" type="fixed">
-    <parent link="base_link"/>
-    <origin rpy="0 0 0" xyz="0 0 ${-wheel_radius}"/>
-    <child  link="base_footprint"/>
-  </joint>
-  <link name="base_footprint">
-  </link>
   <!-- steering-->
-  <xacro:steering_link_macro suffix="steering_front" parent="base_link" x="${wheel_base}" y="0"/>
+  <xacro:steering_link_macro suffix="steering_front" parent="base_body_link" x="${wheel_base}" y="0"/>
   <xacro:steering_macro suffix="steering_right_front" parent="steering_front_link" x="0" y="${-1*wheel_tread/2}" yaw="0" length="${wheel_width}"/>
   <xacro:steering_macro suffix="steering_left_front" parent="steering_front_link" x="0" y="${wheel_tread/2}" yaw="0" length="${wheel_width}"/>
@@ -47,6 +41,6 @@
   <xacro:wheel_macro suffix="wheel_right_front" parent="steering_right_front_link" x="0" y="0" yaw="${pi}" radius="${wheel_radius}" width="${wheel_width}"/>
   <xacro:wheel_macro suffix="wheel_left_front" parent="steering_left_front_link" x="0" y="0" yaw="0" radius="${wheel_radius}" width="${wheel_width}"/>
-  <xacro:wheel_macro suffix="wheel_right_rear" parent="base_link" x="0" y="${-1*wheel_tread/2}" yaw="${pi}" radius="${wheel_radius}" width="${wheel_width}"/>
-  <xacro:wheel_macro suffix="wheel_left_rear" parent="base_link" x="0" y="${wheel_tread/2}" yaw="0" radius="${wheel_radius}" width="${wheel_width}"/>
+  <xacro:wheel_macro suffix="wheel_right_rear" parent="base_body_link" x="0" y="${-1*wheel_tread/2}" yaw="${pi}" radius="${wheel_radius}" width="${wheel_width}"/>
+  <xacro:wheel_macro suffix="wheel_left_rear" parent="base_body_link" x="0" y="${wheel_tread/2}" yaw="0" radius="${wheel_radius}" width="${wheel_width}"/>
   <!-- actuator -->
  	<xacro:include filename="$(find vehicle_model)/urdf/actuator.xacro"/>
